Commit message: Created an SDF-file such that we have ackermann steering with the plugin with joins and links for the steering and driving wheels. This is the base now for controlling the car.

File: src/description/porsche_description.urdf (robot description, URDF)
Before this commit: robot porsche, 2 links, 1 joints
Links:
- added link laser_frame; collision cylinder length=0.04 radius=0.05; visual cylinder length=0.04 radius=0.05
Joints:
- added joint laser_joint: type fixed, parent chassis, child laser_frame, origin xyz=0.1 0 0.175 rpy=0 0 0

Commit message: Finally able to map a room using SLAM where map - odom - base_link.

File: src/description/porsche_description.urdf (robot description, URDF)
Before this commit: robot porsche, 3 links, 2 joints
Joints:
- removed joint base_joint
- added joint base_footprint_joint: type fixed, parent base_link, child base_footprint, origin xyz=0.0 0.0 ${-(wheel_radius+wheel_zoff)} rpy=0 0 0

Commit message: ukf instead of ekf

File: src/description/porsche_description.urdf (robot description, URDF)
Before this commit: robot porsche, 3 links, 2 joints
Joints:
- joint lidar_joint: origin xyz=0 0 0.12 rpy=0 0 0 -> xyz=0 0 0.16 rpy=0 0 0

Commit message: Fixed map -> odom problem

File: src/description/porsche_description.urdf (robot description, URDF)
Before this commit: robot porsche, 3 links, 2 joints
Links:
- removed link lidar_link
- added link laser, mass 0.125; collision cylinder length=0.055 radius=0.0508; visual cylinder length=0.055 radius=0.0508
Joints:
- joint base_footprint_joint: child base_footprint -> base_link; parent base_link -> base_footprint
- joint lidar_joint: child lidar_link -> laser

Commit message: Need Tweeeeeaking

File: src/description/porsche_description.urdf (robot description, URDF)
Before this commit: robot porsche, 3 links, 2 joints
Joints:
- joint base_footprint_joint: child base_link -> base_footprint; origin xyz=0.0 0.0 ${-(wheel_radius+wheel_zoff)} rpy=0 0 0 -> xyz=0.0 0.0 ${-(wheel_radius+wheel_zoff)} rpy=0 0 -1.5708; parent base_footprint -> base_link
- joint lidar_joint: origin xyz=0 0 0.16 rpy=0 0 0 -> xyz=0 0 0.16 rpy=0 0 1.5708

Commit message: It all works now. Just need to perfect all settings

File: src/description/porsche_description.urdf (robot description, URDF)
Before this commit: robot porsche, 3 links, 2 joints
Joints:
- joint lidar_joint: origin xyz=0 0 0.16 rpy=0 0 1.5708 -> xyz=0 0 0.16 rpy=0 0 -1.5708
